Commit message: changed bot colors

File: multi_turtlebots_sim/turtlebot3_description/urdf/turtlebot3_burger.gazebo.xacro (robot description, xacro)
@@ -4,5 +4,5 @@
   <xacro:arg name="imu_visual"   default="false"/>
   <gazebo reference="base_link">
-    <material>Gazebo/DarkGrey</material>
+    <material>Gazebo/Red</material>
   </gazebo>
   <gazebo reference="wheel_left_link">
@@ -14,5 +14,5 @@
     <maxVel>0.1</maxVel>
     <fdir1>1 0 0</fdir1>
-    <material>Gazebo/FlatBlack</material>
+    <material>Gazebo/Blue</material>
   </gazebo>
   <gazebo reference="wheel_right_link">
@@ -24,5 +24,5 @@
     <maxVel>0.1</maxVel>
     <fdir1>1 0 0</fdir1>
-    <material>Gazebo/FlatBlack</material>
+    <material>Gazebo/Blue</material>
   </gazebo>
   <gazebo reference="caster_back_link">
